Commit message: hackery #1

File: gym_gazebo/envs/assets/urdf/erlecopter/erlecopter.xacro (robot description, xacro)
@@ -198,4 +198,11 @@
     <origin xyz="0.17 0.0 0.0" rpy="0 0 0"/>
   </xacro:generic_camera>
+  <!-- Front facing camera -->
+  <xacro:include filename="$(find ardupilot_sitl_gazebo_plugin)/urdf/sensors/kinect.urdf.xacro" />
+  <xacro:generic_camera
+    name="erlecopter/kinect"
+    parent="base_link">
+    <origin xyz="0.17 0.0 0.5" rpy="0 0 0"/>
+  </xacro:generic_camera>
   <!-- Instantiate rotors -->
   <xacro:vertical_rotor
